File: board/rp3802.kicad_pcb (KiCad board)
At the start: 2 copper layers, 57.8 x 61 mm, 14 parts, among them J1 Conn_01x03_Pin, J2 Conn_01x07_Pin, U1 YM3802, U2 Pico

Commit message: changed /IRQ pull up register value.
Parts:
- R1: value 1k -> 10k
Changed lines of the file:
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@@
 			)
 		)
-		(property "Value" "1k"
+		(property "Value" "10k"
 			(at -2.54 1.43 180)
 			(layer "F.Fab")
@@
 	)
 	(zone
-		(net 12)
-		(net_name "/~{IRQ}")
-		(layer "F.Cu")
-		(name "$teardrop_padvia$")
-		(hatch none 0.1)
-		(priority 30031)
-		(attr
-			(teardrop
-				(type padvia)
-			)
-		)
-		(connect_pads yes
-			(clearance 0)
-		)
-		(min_thickness 0.0254)
-		(filled_areas_thickness no)
-		(fill yes
-			(thermal_gap 0.5)
-			(thermal_bridge_width 0.5)
-			(island_removal_mode 1)
-			(island_area_min 10)
-		)
-		(polygon
-			(pts
-				(xy 158.78 74.195) (xy 158.78 74.395) (xy 159.401613 74.751921) (xy 159.7435 74.295) (xy 159.401613 73.838079)
-			)
-		)
-	)
-	(zone
 		(net 1)
 		(net_name "+5V")
@@
 	)
 	(zone
+		(net 12)
+		(net_name "/~{IRQ}")
+		(layer "F.Cu")
+		(name "$teardrop_padvia$")
+		(hatch none 0.1)
+		(priority 30000)
+		(attr
+			(teardrop
+				(type padvia)
+			)
+		)
+		(connect_pads yes
+			(clearance 0)
+		)
+		(min_thickness 0.0254)
+		(filled_areas_thickness no)
+		(fill yes
+			(thermal_gap 0.5)
+			(thermal_bridge_width 0.5)
+			(island_removal_mode 1)
+			(island_area_min 10)
+		)
+		(polygon
+			(pts
+				(xy 158.78 74.195) (xy 158.78 74.395) (xy 159.401613 74.751921) (xy 159.7435 74.295) (xy 159.401613 73.838079)
+			)
+		)
+	)
+	(zone
 		(net 11)
 		(net_name "/GP28")
@@
 	)
 	(zone
+		(net 13)
+		(net_name "/3V3")
+		(layer "F.Cu")
+		(name "$teardrop_padvia$")
+		(hatch none 0.1)
+		(priority 30001)
+		(attr
+			(teardrop
+				(type padvia)
+			)
+		)
+		(connect_pads yes
+			(clearance 0)
+		)
+		(min_thickness 0.0254)
+		(filled_areas_thickness no)
+		(fill yes
+			(thermal_gap 0.5)
+			(thermal_bridge_width 0.5)
+			(island_removal_mode 1)
+			(island_area_min 10)
+		)
+		(polygon
+			(pts
+				(xy 162.53 74.395) (xy 162.53 74.195) (xy 161.908387 73.838079) (xy 161.5665 74.295) (xy 161.908387 74.751921)
+			)
+		)
+	)
+	(zone
 		(net 50)
 		(net_name "/~{CSWR}")
@@
 			)
 		)
-	)
-	(zone
-		(net 13)
-		(net_name "/3V3")
-		(layer "F.Cu")
-		(name "$teardrop_padvia$")
-		(hatch none 0.1)
-		(priority 30035)
-		(attr
-			(teardrop
-				(type padvia)
-			)
-		)
-		(connect_pads yes
-			(clearance 0)
-		)
-		(min_thickness 0.0254)
-		(filled_areas_thickness no)
-		(fill yes
-			(thermal_gap 0.5)
-			(thermal_bridge_width 0.5)
-			(island_removal_mode 1)
-			(island_area_min 10)
-		)
-		(polygon
-			(pts
-				(xy 162.53 74.395) (xy 162.53 74.195) (xy 161.908387 73.838079) (xy 161.5665 74.295) (xy 161.908387 74.751921)
-			)
-		)
