File: board/rp3802.kicad_sch (KiCad schematic)
At the start: 14 parts, among them J1 Conn_01x03_Pin, J2 Conn_01x07_Pin, U1 YM3802, U2 Pico

Commit message: fixed typo in sheet titles.
Other:
- title: RP3803: Tiny YM3802 Emulator by Raspberry Pi Pico -> RP3802: Tiny YM3802 Emulator by Raspberry Pi Pico
- moved on the sheet: D2, D3, D4, D5
Changed lines of the file:
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@@
 	(paper "A4")
 	(title_block
-		(title "RP3803: Tiny YM3802 Emulator by Raspberry Pi Pico")
+		(title "RP3802: Tiny YM3802 Emulator by Raspberry Pi Pico")
 		(date "2025-05-31")
 		(rev "1.0")
@@
 	(symbol
 		(lib_id "Device:LED_Small")
-		(at 73.66 173.99 180)
+		(at 73.66 173.99 0)
+		(mirror y)
 		(unit 1)
 		(exclude_from_sim no)
@@
 		(on_board yes)
 		(dnp no)
-		(fields_autoplaced yes)
 		(property "Reference" "D5"
-			(at 73.5965 167.64 0)
+			(at 73.914 170.942 0)
 			(effects
 				(font
@@
 		)
 		(property "Value" "GP28"
-			(at 73.5965 170.18 0)
+			(at 73.914 168.402 0)
 			(effects
 				(font
@@
 	(symbol
 		(lib_id "Device:LED_Small")
-		(at 73.66 162.56 180)
+		(at 73.66 162.56 0)
+		(mirror y)
 		(unit 1)
 		(exclude_from_sim no)
@@
 		(on_board yes)
 		(dnp no)
-		(fields_autoplaced yes)
 		(property "Reference" "D4"
-			(at 73.5965 156.21 0)
+			(at 73.914 159.258 0)
 			(effects
 				(font
@@
 		)
 		(property "Value" "GP27"
-			(at 73.5965 158.75 0)
+			(at 73.914 156.718 0)
 			(effects
 				(font
@@
 	(symbol
 		(lib_id "Device:LED_Small")
-		(at 73.66 139.7 180)
+		(at 73.66 139.7 0)
+		(mirror y)
 		(unit 1)
 		(exclude_from_sim no)
@@
 		(on_board yes)
 		(dnp no)
-		(fields_autoplaced yes)
 		(property "Reference" "D2"
-			(at 73.5965 133.35 0)
+			(at 73.914 136.144 0)
 			(effects
 				(font
@@
 		)
 		(property "Value" "GP22"
-			(at 73.5965 135.89 0)
+			(at 73.914 133.604 0)
 			(effects
 				(font
@@
 	(symbol
 		(lib_id "Device:LED_Small")
-		(at 73.66 151.13 180)
+		(at 73.66 151.13 0)
+		(mirror y)
 		(unit 1)
 		(exclude_from_sim no)
@@
 		(on_board yes)
 		(dnp no)
-		(fields_autoplaced yes)
 		(property "Reference" "D3"
-			(at 73.5965 144.78 0)
+			(at 73.914 148.082 0)
 			(effects
 				(font
@@
 		)
 		(property "Value" "GP26"
-			(at 73.5965 147.32 0)
+			(at 73.914 145.542 0)
 			(effects
 				(font

Commit message: changed /IRQ pull up register value.
Parts:
- R1: value 1k -> 10k
Changed lines of the file:
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@@
 			)
 		)
-		(property "Value" "1k"
+		(property "Value" "10k"
 			(at 140.97 90.1699 0)
 			(effects
